File: EX-MotorShield8874.kicad_pcb (KiCad board)
At the start: 4 copper layers, 68.6 x 53.3 mm, 101 parts, among them J1 Power, J11 I2C, J12 OLED, J13 MC 1,5/ 2-G-3,5, J14 STEMMA QT, J15 MC 1,5/ 2-G-3,5, J2 Digital/PWM, J3 Analog, J4 Digital/PWM, J51 Barrel_Jack_MountingPin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

Commit message: Replaced the OpAmp comparitor circuit with a single MOSFET.
Parts:
- removed C11, C12: 100nF, Capacitor_SMD:C_0402_1005Metric
- removed R11: 47K, Resistor_SMD:R_0402_1005Metric
- removed R12: 470K, Resistor_SMD:R_0402_1005Metric
- removed U11: LMV321, Package_TO_SOT_SMD:SOT-23-5
- added Q52: BSS84, Package_TO_SOT_SMD:SOT-23, F.Cu at (132.0, 90.5)
- added R56: 47K, Resistor_SMD:R_0402_1005Metric, F.Cu at (131.6, 93.0)
Routing:
- net GND: track 53.2 -> 50.5 mm, vias 68 -> 65
- net /4V5: track 2.67 -> 0.00 mm
- net +5V: track 24.0 -> 21.9 mm
- net VBUS: track 58.0 -> 56.6 mm, vias 13 -> 10
