File: DRV8874.kicad_sch (KiCad schematic)
At the start: 10 parts, among them U104 DRV8874PWPR

Commit message: Stand alone, purpose build command station doodle.
Parts:
- added C103 (x2): 100nF, Capacitor_SMD:C_0402_1005Metric, symbol Device:C_Small
- added J301: ICSP, Connector_PinHeader_2.54mm:PinHeader_1x05_P2.54mm_Vertical, symbol Connector:Conn_01x05_Pin
- added R111: 10K, Resistor_SMD:R_0402_1005Metric, symbol Device:R_Small
- added U302: PIC16F15224-I/ST, Package_SO:TSSOP-14_4.4x5mm_P0.65mm, symbol MCU_Microchip_PIC16:PIC16F1503-IST
- R111: LCSC Part # C25864 -> C25744
Connections:
- net EN/IN1: now also U302.7 (~{SS}/PWM2/CLCIN0/C2IN3-/C1IN3-/AN7/RC3)
- net GND: now also C103.2, C103.2, J301.3 (Pin_3), U302.14 (VSS)
- net PH/IN2: now also U302.6 (CLC2IN1/CWG1B/C2OUT/RC4)
- net VPROPI: now also U302.2 (RA5/T1CKI/NCO1CLK/CLCIN1/CLKIN)
- net VRef: now also C103.1, J301.2 (Pin_2), R111.1, U302.1 (VDD); no longer U104.16 (PMODE), U104.3 (nSleep)
- net nFAULT renamed nFault
- net nFault: now also U302.3 (RA4/AN3/T1G/NCO1/SDO/CLKOUT)
- new net: C103.1, J301.1 (Pin_1), R111.2, U302.4 (RA3/T1G/CLC1IN0/~{SS}/~{MCLR}/Vpp)
- new net: J301.4 (Pin_4), U302.13 (RA0/AN0/DACOUT1/C1IN+/ICSPDAT)
- new net: J301.5 (Pin_5), U302.12 (RA1/AN1/Vref+/C1IN0-/C2IN0-/ICSPCLK)
- new net PMODE: U104.16 (PMODE), U302.8 (SDO/C2IN2-/C1IN2-/AN6/RC2)
- new net SCL: U302.10 (SCK/SCL/CLC2/C2IN+/AN4/RC0)
- new net SDA: U302.9 (SDI/SDA/PWM4/NCO1/C2IN1-/C1IN1-/AN5/RC1)
- new net nSleep: U104.3 (nSleep), U302.5 (PWM1/CLC1/CWG1A/RC5)
