File: EX-MotorShield8874.kicad_sch (KiCad schematic)
At the start: 69 parts, among them J1 Power, J101 MC 1,5/ 2-G-3,5, J103 MC 1,5/ 2-G-3,5, J105 STEMMA QT, J106 I2C, J107 OLED, J2 Digital/PWM, J3 Analog, J4 Digital/PWM, Q101 AO3400A, Q102 AO3400A, Q52 LP2301LT1G, SW101 RESET, U101 74HC04, U102 74HC08, U103 74HC32, U104 DRV8874PWPR, U105 DRV8874PWPR

Commit message: Reworked schematic to include an ESP32-S2-MINI-2.
Reworked schematic to include an ESP32-S2-MINI-2 as the main CPU.

Two track outputs are directly on this board.  The rest of the GPIO
pins are routed so that the existing EX-MotorShield8874 can stack.
The result is potentially 6 power outputs from a single unit.

Added a USB interface to the module.

Moved the drivers into heirarchal sheets.

Removed all unnecessary components.

Added a JTAG header for debugging.
Parts:
- removed C101, C103, C104, C106, C107, C108: 100nF, Capacitor_SMD:C_0402_1005Metric, symbol Device:C_Small
- removed C102, C105: 10uF, Capacitor_SMD:C_0805_2012Metric, symbol Device:C_Small
- removed C109, C110, C112, C113: 22nF, Capacitor_SMD:C_0402_1005Metric, symbol Device:C_Small
- removed C201, C202: 100uF, Capacitor_SMD:CP_Elec_6.3x7.7, symbol Device:C_Polarized_Small
- removed D202: EMERALD, LED_SMD:LED_0603_1608Metric, symbol Device:LED
- removed JP11: PWMA, Jumper:SolderJumper-3_P1.3mm_Bridged12_RoundedPad1.0x1.5mm, symbol Jumper:SolderJumper_3_Bridged12
- removed JP12: BRKA, Jumper:SolderJumper-3_P1.3mm_Bridged12_RoundedPad1.0x1.5mm, symbol Jumper:SolderJumper_3_Bridged12
- removed JP13: PWMB, Jumper:SolderJumper-3_P1.3mm_Bridged12_RoundedPad1.0x1.5mm, symbol Jumper:SolderJumper_3_Bridged12
- removed JP14: BRKB, Jumper:SolderJumper-3_P1.3mm_Bridged12_RoundedPad1.0x1.5mm, symbol Jumper:SolderJumper_3_Bridged12
- removed JP15: DIRB, Jumper:SolderJumper-3_P1.3mm_Bridged12_RoundedPad1.0x1.5mm, symbol Jumper:SolderJumper_3_Bridged12
- removed JP16: DIRA, Jumper:SolderJumper-3_P1.3mm_Bridged12_RoundedPad1.0x1.5mm, symbol Jumper:SolderJumper_3_Bridged12
- removed JP17: FLTA, Jumper:SolderJumper-3_P1.3mm_Bridged12_RoundedPad1.0x1.5mm, symbol Jumper:SolderJumper_3_Bridged12
- removed JP18: FLTB, Jumper:SolderJumper-3_P1.3mm_Bridged12_RoundedPad1.0x1.5mm, symbol Jumper:SolderJumper_3_Bridged12
- removed JP19: SENB, Jumper:SolderJumper-3_P1.3mm_Bridged12_RoundedPad1.0x1.5mm, symbol Jumper:SolderJumper_3_Bridged12
- removed JP20: SENA, Jumper:SolderJumper-3_P1.3mm_Bridged12_RoundedPad1.0x1.5mm, symbol Jumper:SolderJumper_3_Bridged12
- removed JP23: PMODE, Jumper:SolderJumper-3_P1.3mm_Bridged12_RoundedPad1.0x1.5mm, symbol Jumper:SolderJumper_3_Bridged12
- removed JP24: ph/in2a, Jumper:SolderJumper-3_P1.3mm_Bridged12_RoundedPad1.0x1.5mm, symbol Jumper:SolderJumper_3_Bridged12
- removed JP25: nSleepb, Jumper:SolderJumper-3_P1.3mm_Bridged12_RoundedPad1.0x1.5mm, symbol Jumper:SolderJumper_3_Bridged12
- removed JP26: ph/in2b, Jumper:SolderJumper-3_P1.3mm_Bridged12_RoundedPad1.0x1.5mm, symbol Jumper:SolderJumper_3_Bridged12
- removed JP27: nSleepa, Jumper:SolderJumper-3_P1.3mm_Bridged12_RoundedPad1.0x1.5mm, symbol Jumper:SolderJumper_3_Bridged12
- removed JP57: B/P A, Jumper:SolderJumper-3_P1.3mm_Bridged12_RoundedPad1.0x1.5mm, symbol Jumper:SolderJumper_3_Bridged12
- removed JP58: INA, Jumper:SolderJumper-3_P1.3mm_Bridged12_RoundedPad1.0x1.5mm, symbol Jumper:SolderJumper_3_Bridged12
- removed JP59: INB, Jumper:SolderJumper-3_P1.3mm_Bridged12_RoundedPad1.0x1.5mm, symbol Jumper:SolderJumper_3_Bridged12
- removed JP60: B/P B, Jumper:SolderJumper-3_P1.3mm_Bridged12_RoundedPad1.0x1.5mm, symbol Jumper:SolderJumper_3_Bridged12
- removed Q101, Q102: AO3400A, Package_TO_SOT_SMD:SOT-23, symbol Transistor_FET:AO3400A
- removed Q52: LP2301LT1G, Package_TO_SOT_SMD:SOT-23, symbol Transistor_FET:IRF4905
- removed R101, R102, R103, R104, R109, R110, R115, R204: 47K, Resistor_SMD:R_0402_1005Metric, symbol Device:R_Small
- removed R111, R112: 1K43, Resistor_SMD:R_0402_1005Metric, symbol Device:R_Small
- removed R113, R114: 732R, Resistor_SMD:R_0402_1005Metric, symbol Device:R_Small
- removed U101: 74HC04, Package_SO:TSSOP-14_4.4x5mm_P0.65mm, symbol 74xx:74HC04
- removed U102: 74HC08, Package_SO:TSSOP-14_4.4x5mm_P0.65mm, symbol 74xx:74LS08
- removed U103: 74HC32, Package_SO:TSSOP-14_4.4x5mm_P0.65mm, symbol 74xx:74LS32
- removed U104, U105: DRV8874PWPR, Package_SO:HTSSOP-16-1EP_4.4x5mm_P0.65mm_EP3.4x5mm_Mask2.46x2.31mm_ThermalVias, symbol DCC-EX-Symbols:DRV8874PWPR
- added C103 (x4): 20pF, Capacitor_SMD:C_0402_1005Metric, symbol Device:C_Small
- added J101: USB_B_Micro, Connector_USB:USB_Micro-B_Molex-105017-0001, symbol Connector:USB_B_Micro
- added J102: JTAG, Connector_PinHeader_2.54mm:PinHeader_2x05_P2.54mm_Vertical, symbol Connector_Generic:Conn_02x05_Odd_Even
- added U52: ESP32-S2-MINI-1, PCM_Espressif:ESP32-S2-MINI-1, symbol PCM_Espressif:ESP32-S2-MINI-1
- added Y101: 40Mhz, Crystal:Crystal_SMD_7050-4Pin_7.0x5.0mm, symbol Device:Crystal_GND24_Small
- SW101: value RESET -> FLASH
Connections:
- net IOREF is gone; now on net +3V3: J1.2 (Pin_2)
- net VBUS is gone; now on net +3V3: J106.1 (Pin_1), J106.2 (Pin_2), J107.2 (Pin_2)
- net +3V3: now also J102.1 (Pin_1), U52.3 (3V3)
- net GND: now also C103.2, C103.2, C103.2, C103.2, J101.4 (ID), J101.5 (GND), J101.6 (Shield), U52.1 (GND), U52.2 (GND), U52.30 (GND), U52.42 (GND), U52.43 (GND), U52.46 (GND), U52.47 (GND), U52.48 (GND), U52.49 (GND), U52.50 (GND), U52.51 (GND), U52.52 (GND), U52.53 (GND), U52.54 (GND), U52.55 (GND), U52.56 (GND), U52.57 (GND), U52.58 (GND), U52.59 (GND), U52.60 (GND), U52.61 (GND), U52.62 (GND), U52.63 (GND), U52.64 (GND), U52.65 (GND), Y101.2, Y101.4
- net alt_brake_a: now also U52.18 (GPIO14/ADC2_CH3)
- net alt_brake_b: now also U52.33 (GPIO37)
- net alt_direction_a: now also U52.16 (GPIO12/ADC2_CH1)
- net alt_direction_b: now also U52.31 (GPIO35)
- net alt_fault_n_a: now also U52.22 (ADC2_CH6/DAC_1/GPIO18)
- net alt_fault_n_b: now also U52.41 (GPIO45)
- net alt_pwm_a: now also U52.14 (GPIO10/ADC1_CH9)
- net alt_pwm_b: now also U52.28 (GPIO33)
- net alt_sen_a: now also U52.8 (GPIO4/ADC1_CH3)
- net alt_sen_b: now also U52.10 (GPIO6/ADC1_CH5)
- net def_brake_a: now also U52.17 (GPIO13/ADC2_CH2)
- net def_brake_b: now also U52.32 (GPIO36)
- net def_direction_a: now also U52.15 (GPIO11/ADC2_CH0)
- net def_direction_b: now also U52.29 (GPIO34)
- net def_fault_n_a: now also U52.21 (ADC2_CH7/DAC_2/GPIO17)
- net def_fault_n_b: now also U52.34 (GPIO38)
- net def_pwm_a: now also U52.13 (GPIO9/ADC1_CH8)
- net def_pwm_b: now also U52.25 (GPIO21)
- net def_sen_a: now also U52.7 (GPIO3/ADC1_CH2)
- net def_sen_b: now also U52.9 (GPIO5/ADC1_CH4)
- net +5V: no longer names the net of J1.5 (Pin_5)
- net VCOM: no longer names the net of J1.8 (Pin_8)
- net reset: no longer names the net of J1.3 (Pin_3)
- net reset: no longer SW101.1
- new net: C103.1, U52.19 (GPIO15/ADC2_CH4/XTAL_32K_P), Y101.3
- new net: C103.1, U52.20 (GPIO16/ADC2_CH5/XTAL_32K_N), Y101.1
- new net: J102.3 (Pin_3), J102.5 (Pin_5), J102.9 (Pin_9)
- new net BOOT_MODE: SW101.1, U52.4 (GPIO0/BOOT)
- new net Out1-IN1: U52.11 (GPIO7/ADC1_CH6)
- new net Out1-IN2: U52.12 (GPIO8/ADC1_CH7)
- new net Out1-Vpropi: U52.5 (GPIO1/ADC1_CH0)
- new net Out2-IN1: U52.44 (GPIO46)
- new net Out2-IN2: U52.26 (SPI_CS1/GPIO26)
- new net Out2-Vpropi: U52.6 (GPIO2/ADC1_CH1)
- new net TCK: J102.4 (Pin_4), U52.35 (MTCK/JTAG/GPIO39)
- new net TDI: J102.8 (Pin_8), U52.37 (MTDI/JTAG/GPIO41)
- new net TDO: J102.6 (Pin_6), U52.36 (MTDO/JTAG/GPIO40)
- new net TMS: J102.2 (Pin_2), U52.38 (MTMS/JTAG/GPIO42)
- new net USB_D+: C103.1, J101.3 (D+), U52.24 (USB_D+/ADC2_CH9/GPIO20)
- new net USB_D-: C103.1, J101.2 (D-), U52.23 (USB_D-/ADC2_CH8/GPIO19)
- new net ~{SRST}: J102.10 (Pin_10), U52.45 (CHIP/PU/RESET)
- no-connect marks 4 -> 9
Other:
- added sheet Output 1 (DRV8874.kicad_sch)
- added sheet Output 2 (DRV8874.kicad_sch)
- sheet Power ports: added 3V3-Out; removed none
- note added: "3V3"
- note added: "5V"
- note added: "Buck Converter Power Supply"
- note added: "Expose RS232 Serial? Use for sda/scl I2C bus?"
- note added: "IOREF"
- note added: "Motor Drivers"
- note added: "Output Indicators Red/Green LEDs"
- note added: "RESET"
- note added: "VIN"
- note removed: "* Indicates a PWM-capable pin"
- note removed: "Alternative pinout to allow stacking"
- note removed: "Channel A Defaults: D12 - Direction D3 - PWM (work duty) D9 - Brake A0 - current sensing."
- note removed: "Channel B Defaults: D13 - Direction D11 - PWM (work duty) D8 - Brake A1 - current sensing"
- note removed: "Configuration Logic"
- note removed: "DRV8874 (max 6A) Current Sensing: V_prop is limited to VRef inside DRV8874 5V = 0.000455*(1430+732)*A => A=5,08 3,3V = 0.000455* 1430 *A => A=5,07 if subbed with DRV8876 (max 3.5A): 5V = 0.001*(x+y)*A => A= 3,3V = 0.001* x *A => A="
- note removed: "DRV8874 Mode Select"
- note removed: "DRV8874 Motor Drivers"
- note removed: "If VBUS (IOREF) is 5V, Vgs = 0V, the PMOS is off, VBUS_is_3V3_not_5V will be pulled down to ground by R11. If VBUS (IOREF) is 3.3V, Vgs = -1.7V, the PMOS is on, VBUS_is_3V3_not_5V will be connected to +5V. Downstream the two NMOS will get a signal of 0, or +5V. A Vgs of +5V will fully turn them on, even though the drain voltage is only 3.3V."
- note removed: "Indicators"
- note removed: "LP2301LT1G has Vgs(th) = 0.9V. A BSS84 will likely work, but some have Vgs(th) of 1.7V which leaves no margin."
- note removed: "PH/EN Mode (PMODE Low) nSleep/EN/PH out1/2 0 X X ZZ 1 0 X 00 1 1 0 01 1 1 1 10 nSleep = high / pwm EN = not brake / pwm PH = dir"
- note removed: "PWM Mode (PMODE High) nSleep/in1/2 out1/2 O X X ZZ 1 0 0 ZZ 1 0 1 01 1 1 0 10 1 1 1 00 nSleep = high in1 = pwm and ( dir or brake) in2 = pwm and (not dir or brake)"
- note removed: "Power Sheet"
- note removed: "VBUS Voltage Determination"
- note removed: "candidate values: 2k+1k 3.63/1.65 1% 1k8+(680+220) 4.0/1.83 1% 1k5+(680+100) 4.8/2.2 0.2% 1k43+732(extend.) 5.08 0.1% <-- USED HERE (1k2+120)+680 5.5/2.5 0.0% 1k2+(470+180) 5.9/2.7 2% 1k2+620(extend.) 5.9/2.7 0.1% 1k1+560 (0603) 6.6/3.0 0.4%"
- note removed: "n_channel conducts if gate high"
- moved on the sheet: D54, D55, J101, J103, J107, R204

Commit message: Update BOM to include all parts.
Parts:
- J105: renamed from J102; LCSC Part # (none) -> C2935920
- J109: renamed from J101; LCSC Part # (none) -> C136000
- U101: renamed from U52; value ESP32-S2-MINI-1 -> ESP32-S2-MINI-2; LCSC Part # (none) -> C3013906; MPN (none) -> ESP32-S2-MINI-2-N4; Manufacturer (none) -> Espressif; Substitute (none) -> No; rohs_cert_or_in_datasheet (none) -> y
- Y101: footprint Crystal:Crystal_SMD_7050-4Pin_7.0x5.0mm -> Crystal:Crystal_SMD_5032-4Pin_5.0x3.2mm; LCSC Part # (none) -> C2901643
- renumbered D54 to D101, D55 to D102, J2 to J104, J1 to J106, J3 to J110, J4 to J111

Commit message: Initial attempt to route the board.
Parts:
- renumbered J106 to J101, J110 to J102, J104 to J103, J111 to J104, J109 to J108, J105 to J111
Connections:
- net GND: now also J111.3 (Pin_3), J111.5 (Pin_5), J111.9 (Pin_9)
- net alt_sen_a: now also U101.9 (GPIO5/ADC1_CH4); no longer U101.8 (GPIO4/ADC1_CH3)
- net alt_sen_b: now also U101.7 (GPIO3/ADC1_CH2); no longer U101.10 (GPIO6/ADC1_CH5)
- net def_sen_a: now also U101.10 (GPIO6/ADC1_CH5); no longer U101.7 (GPIO3/ADC1_CH2)
- net def_sen_b: now also U101.8 (GPIO4/ADC1_CH3); no longer U101.9 (GPIO5/ADC1_CH4)
Changed lines of the file:
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@@
   (junction (at 157.48 74.93) (diameter 0) (color 0 0 0 0)
+  )
+  (junction (at 232.41 55.88) (diameter 0) (color 0 0 0 0)
   )
   (junction (at 161.29 85.09) (diameter 0) (color 0 0 0 0)
@@
     (stroke (width 0) (type default))
   )
+  (wire (pts (xy 232.41 55.88) (xy 232.41 58.42))
+    (stroke (width 0) (type default))
+  )
   (wire (pts (xy 81.28 60.96) (xy 93.98 60.96))
     (stroke (width 0) (type solid))
@@
     (effects (font (size 1.27 1.27)) (justify left bottom))
   )
-  (label "trk2l" (at 243.84 200.66 0) (fields_autoplaced)
+  (label "trk2l" (at 243.84 205.74 0) (fields_autoplaced)
     (effects (font (size 1.27 1.27)) (justify left bottom))
   )
@@
     (effects (font (size 1.27 1.27)) (justify right bottom))
   )
-  (label "trk1l" (at 243.84 149.86 0) (fields_autoplaced)
+  (label "trk1l" (at 243.84 154.94 0) (fields_autoplaced)
     (effects (font (size 1.27 1.27)) (justify left bottom))
   )
@@
     (effects (font (size 1.27 1.27)) (justify right bottom))
   )
-  (label "alt_sen_a" (at 134.62 165.1 0) (fields_autoplaced)
+  (label "alt_sen_a" (at 134.62 167.64 0) (fields_autoplaced)
     (effects (font (size 1.27 1.27)) (justify left bottom))
   )
@@
     (effects (font (size 1.27 1.27)) (justify right bottom))
   )
-  (label "alt_sen_b" (at 134.62 170.18 0) (fields_autoplaced)
+  (label "alt_sen_b" (at 134.62 162.56 0) (fields_autoplaced)
     (effects (font (size 1.27 1.27)) (justify left bottom))
   )
@@
     (effects (font (size 1.27 1.27)) (justify left bottom))
   )
-  (label "trk1r" (at 243.84 154.94 0) (fields_autoplaced)
+  (label "trk1r" (at 243.84 149.86 0) (fields_autoplaced)
     (effects (font (size 1.27 1.27)) (justify left bottom))
   )
@@
     (effects (font (size 1.27 1.27)) (justify left bottom))
   )
-  (label "trk2r" (at 243.84 205.74 0) (fields_autoplaced)
-    (effects (font (size 1.27 1.27)) (justify left bottom))
-  )
-  (label "def_sen_a" (at 134.62 162.56 0) (fields_autoplaced)
+  (label "trk2r" (at 243.84 200.66 0) (fields_autoplaced)
+    (effects (font (size 1.27 1.27)) (justify left bottom))
+  )
+  (label "def_sen_a" (at 134.62 170.18 0) (fields_autoplaced)
     (effects (font (size 1.27 1.27)) (justify left bottom))
   )
@@
     (effects (font (size 1.27 1.27)) (justify left bottom))
   )
-  (label "def_sen_b" (at 134.62 167.64 0) (fields_autoplaced)
+  (label "def_sen_b" (at 134.62 165.1 0) (fields_autoplaced)
     (effects (font (size 1.27 1.27)) (justify left bottom))
   )
@@
   (symbol (lib_id "Connector_Generic:Conn_01x08") (at 57.15 53.34 0) (unit 1)
     (in_bom yes) (on_board yes) (dnp no)
-    (property "Reference" "J106" (at 57.15 43.18 0)
+    (property "Reference" "J101" (at 57.15 43.18 0)
       (effects (font (size 1.27 1.27)))
     )
@@
       (project "EX-MotorShield8874"
         (path "/e63e39d7-6ac0-4ffd-8aa3-1841a4541b55"
-          (reference "J106") (unit 1)
+          (reference "J101") (unit 1)
         )
       )
@@
   (symbol (lib_id "Connector_Generic:Conn_01x10") (at 76.2 50.8 0) (mirror y) (unit 1)
     (in_bom yes) (on_board yes) (dnp no)
-    (property "Reference" "J104" (at 76.2 38.1 0)
+    (property "Reference" "J103" (at 76.2 38.1 0)
       (effects (font (size 1.27 1.27)))
     )
@@
       (project "EX-MotorShield8874"
         (path "/e63e39d7-6ac0-4ffd-8aa3-1841a4541b55"
-          (reference "J104") (unit 1)
+          (reference "J103") (unit 1)
         )
       )
@@
   (symbol (lib_id "Connector_Generic:Conn_01x06") (at 57.15 81.28 0) (unit 1)
     (in_bom yes) (on_board yes) (dnp no)
-    (property "Reference" "J110" (at 57.15 73.66 0)
+    (property "Reference" "J102" (at 57.15 73.66 0)
       (effects (font (size 1.27 1.27)))
     )
@@
       (project "EX-MotorShield8874"
         (path "/e63e39d7-6ac0-4ffd-8aa3-1841a4541b55"
-          (reference "J110") (unit 1)
+          (reference "J102") (unit 1)
         )
       )
@@
   (symbol (lib_id "Connector_Generic:Conn_01x08") (at 76.2 83.82 0) (mirror y) (unit 1)
     (in_bom yes) (on_board yes) (dnp no)
-    (property "Reference" "J111" (at 76.2 73.66 0)
+    (property "Reference" "J104" (at 76.2 73.66 0)
       (effects (font (size 1.27 1.27)))
     )
@@
       (project "EX-MotorShield8874"
         (path "/e63e39d7-6ac0-4ffd-8aa3-1841a4541b55"
-          (reference "J111") (unit 1)
+          (reference "J104") (unit 1)
         )
       )
@@
       (project "EX-MotorShield8874"
         (path "/e63e39d7-6ac0-4ffd-8aa3-1841a4541b55"
-          (reference "J101") (unit 1)
+          (reference "J109") (unit 1)
         )
       )
@@
       (project "EX-MotorShield8874"
         (path "/e63e39d7-6ac0-4ffd-8aa3-1841a4541b55"
-          (reference "J108") (unit 1)
+          (reference "J106") (unit 1)
         )
       )
@@
       (project "EX-MotorShield8874"
         (path "/e63e39d7-6ac0-4ffd-8aa3-1841a4541b55"
-          (reference "C101") (unit 1)
+          (reference "C105") (unit 1)
         )
       )
@@
       (project "EX-MotorShield8874"
         (path "/e63e39d7-6ac0-4ffd-8aa3-1841a4541b55"
-          (reference "J103") (unit 1)
+          (reference "J107") (unit 1)
         )
       )
@@
       (project "EX-MotorShield8874"
         (path "/e63e39d7-6ac0-4ffd-8aa3-1841a4541b55"
-          (reference "C103") (unit 1)
+          (reference "C104") (unit 1)
         )
         (path "/e63e39d7-6ac0-4ffd-8aa3-1841a4541b55/fa2ff518-4097-4d36-81d9-67cd6f2fe7e8"
@@
   (symbol (lib_id "Connector:USB_B_Micro") (at 179.07 74.93 0) (mirror y) (unit 1)
     (in_bom yes) (on_board yes) (dnp no) (fields_autoplaced)
-    (property "Reference" "J109" (at 185.42 73.66 0)
+    (property "Reference" "J108" (at 185.42 73.66 0)
       (effects (font (size 1.27 1.27)) (justify right))
     )
@@
       (project "EX-MotorShield8874"
         (path "/e63e39d7-6ac0-4ffd-8aa3-1841a4541b55"
-          (reference "J109") (unit 1)
+          (reference "J108") (unit 1)
         )
       )
@@
       (project "EX-MotorShield8874"
         (path "/e63e39d7-6ac0-4ffd-8aa3-1841a4541b55"
-          (reference "J107") (unit 1)
+          (reference "J110") (unit 1)
         )
       )
@@
       (project "EX-MotorShield8874"
         (path "/e63e39d7-6ac0-4ffd-8aa3-1841a4541b55"
-          (reference "C105") (unit 1)
+          (reference "C102") (unit 1)
         )
         (path "/e63e39d7-6ac0-4ffd-8aa3-1841a4541b55/fa2ff518-4097-4d36-81d9-67cd6f2fe7e8"
@@
       (project "EX-MotorShield8874"
         (path "/e63e39d7-6ac0-4ffd-8aa3-1841a4541b55"
-          (reference "J102") (unit 1)
+          (reference "J105") (unit 1)
         )
       )
@@
   (symbol (lib_id "Connector_Generic:Conn_02x05_Odd_Even") (at 240.03 50.8 0) (unit 1)
     (in_bom yes) (on_board yes) (dnp no) (fields_autoplaced)
-    (property "Reference" "J105" (at 241.3 39.37 0)
+    (property "Reference" "J111" (at 241.3 39.37 0)
       (effects (font (size 1.27 1.27)))
     )
@@
       (project "EX-MotorShield8874"
         (path "/e63e39d7-6ac0-4ffd-8aa3-1841a4541b55"
-          (reference "J105") (unit 1)
+          (reference "J111") (unit 1)
         )
       )
@@
       (project "EX-MotorShield8874"
         (path "/e63e39d7-6ac0-4ffd-8aa3-1841a4541b55"
-          (reference "C104") (unit 1)
+          (reference "C101") (unit 1)
         )
         (path "/e63e39d7-6ac0-4ffd-8aa3-1841a4541b55/fa2ff518-4097-4d36-81d9-67cd6f2fe7e8"
@@
       (project "EX-MotorShield8874"
         (path "/e63e39d7-6ac0-4ffd-8aa3-1841a4541b55"
-          (reference "C102") (unit 1)
+          (reference "C103") (unit 1)
         )
         (path "/e63e39d7-6ac0-4ffd-8aa3-1841a4541b55/fa2ff518-4097-4d36-81d9-67cd6f2fe7e8"
@@
         )
       )
+    )
+  )
+  (symbol (lib_id "power:GND") (at 232.41 58.42 0) (unit 1)
+    (in_bom yes) (on_board yes) (dnp no) (fields_autoplaced)
+    (property "Reference" "#PWR0137" (at 232.41 64.77 0)
+      (effects (font (size 1.27 1.27)) hide)
+    )
+    (property "Value" "GND" (at 232.41 63.5 0)
+      (effects (font (size 1.27 1.27)))
+    )
+    (property "Footprint" "" (at 232.41 58.42 0)
+      (effects (font (size 1.27 1.27)) hide)
+    )
+    (property "Datasheet" "" (at 232.41 58.42 0)
+      (effects (font (size 1.27 1.27)) hide)
+    )
+    (pin "1")
+    (instances
+      (project "motor-shield"
+        (path "/0cbffc97-6856-4b34-94fa-39a0ff6f1c2b"
+          (reference "#PWR0137") (unit 1)
+        )
+      )
+      (project "EX-MotorShield8874"
+        (path "/e63e39d7-6ac0-4ffd-8aa3-1841a4541b55"
+          (reference "#PWR0123") (unit 1)
+        )
+      )
